File: Whale_Lamp-base.brd (EAGLE design)
At the start: 125 x 125 mm, 91 parts, among them Q2 20mA/30V, Q3 16MHz, Q5 2.5A/30V/105mΩ, U0 32U4

Commit message: finished board layout
Parts:
- moved R_OC 48.5 mm to (-11.9, 0.02), turned to 0 degrees
- moved R_SCL 47.8 mm to (7.50, -14.5), turned to 0 degrees
- moved L3 47.1 mm to (-7.00, 7.50), turned to 0 degrees
- moved R_SDA 47.0 mm to (7.50, -12.5), turned to 0 degrees
- moved FP6291 45.0 mm to (-11.9, 3.02), turned to 180 degrees
- moved D_BOOST 43.0 mm to (-7.50, 11.5), turned to 0 degrees
- moved C15 42.4 mm to (-1.03, 9.98), turned to 270 degrees
- moved C13 42.1 mm to (-3.13, 9.98), turned to 270 degrees
- moved R1_BOOST 42.1 mm to (-10.8, 8.90), turned to 90 degrees
- moved C12 41.8 mm to (-15.0, 6.30), turned to 180 degrees
- moved C19 41.6 mm to (-1.03, 13.0), turned to 90 degrees
- moved C18 41.4 mm to (-3.13, 13.0), turned to 90 degrees
- moved C7 39.9 mm to (-15.0, 4.70), turned to 180 degrees
- moved R2_BOOST 39.5 mm to (-12.9, 8.90), turned to 270 degrees
- moved C6 37.5 mm to (-15.0, 2.60), turned to 180 degrees
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Connections:
- removed net 3.3V: CORTEX_SWD1.4
- net 5V: now also CORTEX_SWD1.4
Routing:
- net 5V: track 51.2 -> 848.7 mm, vias 0 -> 40
- net LED_G: track 44.6 -> 545.2 mm, vias 0 -> 34
- net SDA: track 0.00 -> 63.7 mm, vias 0 -> 2
- net SCL: track 0.00 -> 62.3 mm, vias 0 -> 2
- net SS_TX: track 2.60 -> 59.6 mm, vias 0 -> 1
- net SS_RX: track 2.60 -> 59.4 mm, vias 0 -> 1
- net D-: track 0.00 -> 54.1 mm, vias 0 -> 2
- net D+: track 0.00 -> 53.9 mm, vias 0 -> 2
- net N$29: track 0.00 -> 26.1 mm
- net LED_DOUT: track 2.81 -> 28.3 mm, vias 0 -> 2
- net N$38: track 0.00 -> 25.0 mm
- net N$49: track 0.00 -> 23.9 mm
- net N$13: track 0.00 -> 21.1 mm
- net MISO: track 0.00 -> 19.0 mm, vias 0 -> 1
- net 9V: track 4.97 -> 22.4 mm
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
Commit message: Silkscreen cleanup and added additional info into schematic
Parts:
- IR_LED: value (none) -> IR
- PWR_LED: value (none) -> ORANGE
- R_IRLED: value 190 -> 200; device adafruit:R0402 -> adafruit:R0603
- R_SCL, R_SDA: value 510 -> 2.2K
- USER_LED: value (none) -> BLUE
- moved J1 0.71 mm to (-61.2, 0.10)
- moved R_IRLED 0.50 mm to (5.50, 0.00), turned to 90 degrees
Connections:
- net IR_LED: now also R_IRLED.1; no longer R_IRLED.2
- net N$48: now also R_IRLED.2; no longer R_IRLED.1
Routing:
- net D-: track 54.1 -> 55.3 mm
- net D+: track 53.9 -> 55.2 mm
- net N$53: track 2.01 -> 2.75 mm
- net N$51: track 2.03 -> 2.69 mm
- net N$48: track 1.54 -> 2.04 mm
