File: Whale_Lamp-jlc-v2.brd (EAGLE design)
At the start: 29 x 29 mm, 45 parts, among them Q3 16MHz, U0 32U4, U1 MCP73831, U2 FXOS8700CQR1

Commit message: JLC_Order_11-24-2020
Parts:
- C16, C17: value 18pF -> 12pF
- Q3: value 16MHz -> 8MHz
Connections:
- net PC7 renamed SS_RX
- net POW_LED renamed SS_TX
- new net G1: Q3.4
- new net G2: Q3.2
- net GND: no longer Q3.2, Q3.4
Routing:
- net SS_TX: track 0.00 -> 1.87 mm, vias 0 -> 1
- net SS_RX: track 0.00 -> 1.46 mm, vias 0 -> 1
- net ACC_RST: track 26.0 -> 25.0 mm
- net SCL: track 14.7 -> 13.7 mm
- net GND: track 27.4 -> 26.9 mm
Other:
- board text added: "V2"
