File: Whale_Lamp-jlc-v2.sch (EAGLE design)
At the start: 45 parts, among them Q3 16MHz, U0 32U4, U1 MCP73831, U2 FXOS8700CQR1

Commit message: JLC_Order_11-24-2020
Parts:
- C16, C17: value 18pF -> 12pF
- Q3: value 16MHz -> 8MHz
Connections:
- net PC7 renamed SS_RX
- net POW_LED renamed SS_TX
- net GND: no longer Q3.G1, Q3.G2
Changed lines of the file:
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@@
 <?xml version="1.0" encoding="utf-8"?>
 <!DOCTYPE eagle SYSTEM "eagle.dtd">
-<eagle version="9.6.2">
+<eagle version="8.3.1">
 <drawing>
 <settings>
@@
 <part name="FRAME1" library="frames" library_urn="urn:adsk.eagle:library:229" deviceset="DINA3_L" device=""/>
 <part name="GND6" library="SparkFun-Aesthetics" deviceset="GND" device=""/>
-<part name="C16" library="SparkFun" deviceset="CAP" device="0402-CAP" value="18pF"/>
-<part name="C17" library="SparkFun" deviceset="CAP" device="0402-CAP" value="18pF"/>
+<part name="C16" library="SparkFun" deviceset="CAP" device="0402-CAP" value="12pF"/>
+<part name="C17" library="SparkFun" deviceset="CAP" device="0402-CAP" value="12pF"/>
 <part name="GND29" library="SparkFun" deviceset="GND" device=""/>
 <part name="CORTEX_SWD1" library="samd21-temp" deviceset="CORTEX_DEBUG" device="PTH" value="CORTEX_DEBUGPTH"/>
@@
 <part name="R_D-" library="adafruit" deviceset="R-US_" device="R0402" value="22"/>
 <part name="GND10" library="SparkFun-Aesthetics" deviceset="GND" device=""/>
-<part name="Q3" library="adafruit" deviceset="XTAL-4" device="-3225" value="16MHz"/>
+<part name="Q3" library="adafruit" deviceset="XTAL-4" device="-3225" value="8MHz"/>
 <part name="R_LED" library="adafruit" deviceset="R-US_" device="R0402" value="510"/>
 <part name="SUPPLY4" library="SparkFun-PowerSymbols" deviceset="3.3V" device=""/>
@@
 <wire x1="-81.28" y1="-236.22" x2="-81.28" y2="-238.76" width="0.1524" layer="91"/>
 <junction x="-81.28" y="-236.22"/>
-<pinref part="Q3" gate="G$1" pin="G2"/>
-<wire x1="-68.58" y1="-223.52" x2="-81.28" y2="-223.52" width="0.1524" layer="91"/>
-<wire x1="-81.28" y1="-223.52" x2="-81.28" y2="-220.98" width="0.1524" layer="91"/>
 <pinref part="C16" gate="G$1" pin="1"/>
 <wire x1="-81.28" y1="-220.98" x2="-78.74" y2="-220.98" width="0.1524" layer="91"/>
-<wire x1="-81.28" y1="-236.22" x2="-81.28" y2="-233.68" width="0.1524" layer="91"/>
-<junction x="-81.28" y="-223.52"/>
-<pinref part="Q3" gate="G$1" pin="G1"/>
-<wire x1="-81.28" y1="-233.68" x2="-81.28" y2="-223.52" width="0.1524" layer="91"/>
-<wire x1="-68.58" y1="-233.68" x2="-81.28" y2="-233.68" width="0.1524" layer="91"/>
-<junction x="-81.28" y="-233.68"/>
+<wire x1="-81.28" y1="-236.22" x2="-81.28" y2="-220.98" width="0.1524" layer="91"/>
 </segment>
 <segment>
@@
 </segment>
 </net>
-<net name="PC7" class="0">
-<segment>
-<wire x1="-17.78" y1="-236.22" x2="-7.62" y2="-236.22" width="0.1524" layer="91"/>
+<net name="SS_RX" class="0">
+<segment>
+<wire x1="-17.78" y1="-236.22" x2="5.08" y2="-236.22" width="0.1524" layer="91"/>
 <label x="-15.24" y="-236.22" size="1.778" layer="95"/>
 <pinref part="U0" gate="G$1" pin="PC7"/>
+<label x="5.08" y="-236.22" size="1.27" layer="95" xref="yes"/>
 </segment>
 </net>
@@
 </segment>
 </net>
-<net name="POW_LED" class="0">
+<net name="SS_TX" class="0">
 <segment>
 <label x="-15.24" y="-215.9" size="1.778" layer="95"/>
